File: ArduinoPCB.sch (EAGLE design)
At the start: 1 part

Commit message: added pcb
Parts:
- added LED1, LED2, LED3: (no value), led:LED3MM
- added R1, R2, R3, R4: (no value), rcl:R-US_0309/12
- added S5, S6, S7, S8: (no value), switch-dil:DS01E
Connections:
- new net N$1: R4.1, S8.2
- new net N$2: R3.1, S7.2
- new net N$3: R2.1, S6.2
- new net N$4: R1.1, S5.2
Changed lines of the file:
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@@
 <parts>
 <part name="FRAME1" library="SparkFun-Aesthetics" library_urn="urn:adsk.eagle:library:507" deviceset="FRAME-LETTER" device="" package3d_urn="urn:adsk.eagle:package:37121/1"/>
+<part name="LED1" library="led" library_urn="urn:adsk.eagle:library:259" deviceset="LED" device="3MM" package3d_urn="urn:adsk.eagle:package:15797/1"/>
+<part name="LED2" library="led" library_urn="urn:adsk.eagle:library:259" deviceset="LED" device="3MM" package3d_urn="urn:adsk.eagle:package:15797/1"/>
+<part name="LED3" library="led" library_urn="urn:adsk.eagle:library:259" deviceset="LED" device="3MM" package3d_urn="urn:adsk.eagle:package:15797/1"/>
+<part name="R1" library="rcl" library_urn="urn:adsk.eagle:library:334" deviceset="R-US_" device="0309/12" package3d_urn="urn:adsk.eagle:package:23571/1"/>
+<part name="R2" library="rcl" library_urn="urn:adsk.eagle:library:334" deviceset="R-US_" device="0309/12" package3d_urn="urn:adsk.eagle:package:23571/1"/>
+<part name="R3" library="rcl" library_urn="urn:adsk.eagle:library:334" deviceset="R-US_" device="0309/12" package3d_urn="urn:adsk.eagle:package:23571/1"/>
+<part name="R4" library="rcl" library_urn="urn:adsk.eagle:library:334" deviceset="R-US_" device="0309/12" package3d_urn="urn:adsk.eagle:package:23571/1"/>
+<part name="S5" library="switch-dil" library_urn="urn:adsk.eagle:library:375" deviceset="DS01E" device="" package3d_urn="urn:adsk.eagle:package:27201/2"/>
+<part name="S6" library="switch-dil" library_urn="urn:adsk.eagle:library:375" deviceset="DS01E" device="" package3d_urn="urn:adsk.eagle:package:27201/2"/>
+<part name="S7" library="switch-dil" library_urn="urn:adsk.eagle:library:375" deviceset="DS01E" device="" package3d_urn="urn:adsk.eagle:package:27201/2"/>
+<part name="S8" library="switch-dil" library_urn="urn:adsk.eagle:library:375" deviceset="DS01E" device="" package3d_urn="urn:adsk.eagle:package:27201/2"/>
 </parts>
 <sheets>
@@
 <attribute name="DRAWING_NAME" x="157.734" y="5.08" size="2.7432" layer="94" font="vector"/>
 </instance>
+<instance part="LED1" gate="G$1" x="15.24" y="149.86" smashed="yes">
+<attribute name="NAME" x="18.796" y="145.288" size="1.778" layer="95" rot="R90"/>
+<attribute name="VALUE" x="20.955" y="145.288" size="1.778" layer="96" rot="R90"/>
+</instance>
+<instance part="LED2" gate="G$1" x="15.24" y="129.54" smashed="yes">
+<attribute name="NAME" x="18.796" y="124.968" size="1.778" layer="95" rot="R90"/>
+<attribute name="VALUE" x="20.955" y="124.968" size="1.778" layer="96" rot="R90"/>
+</instance>
+<instance part="LED3" gate="G$1" x="15.24" y="109.22" smashed="yes">
+<attribute name="NAME" x="18.796" y="104.648" size="1.778" layer="95" rot="R90"/>
+<attribute name="VALUE" x="20.955" y="104.648" size="1.778" layer="96" rot="R90"/>
+</instance>
+<instance part="R1" gate="G$1" x="30.48" y="88.9" smashed="yes">
+<attribute name="NAME" x="26.67" y="90.3986" size="1.778" layer="95"/>
+<attribute name="VALUE" x="26.67" y="85.598" size="1.778" layer="96"/>
+</instance>
+<instance part="R2" gate="G$1" x="30.48" y="71.12" smashed="yes">
+<attribute name="NAME" x="26.67" y="72.6186" size="1.778" layer="95"/>
+<attribute name="VALUE" x="26.67" y="67.818" size="1.778" layer="96"/>
+</instance>
+<instance part="R3" gate="G$1" x="33.02" y="55.88" smashed="yes">
+<attribute name="NAME" x="29.21" y="57.3786" size="1.778" layer="95"/>
+<attribute name="VALUE" x="29.21" y="52.578" size="1.778" layer="96"/>
+</instance>
+<instance part="R4" gate="G$1" x="30.48" y="35.56" smashed="yes">
+<attribute name="NAME" x="26.67" y="37.0586" size="1.778" layer="95"/>
+<attribute name="VALUE" x="26.67" y="32.258" size="1.778" layer="96"/>
+</instance>
+<instance part="S5" gate="1" x="15.24" y="83.82" smashed="yes">
+<attribute name="NAME" x="17.78" y="80.01" size="1.778" layer="95" rot="R90"/>
+<attribute name="VALUE" x="20.32" y="80.01" size="1.778" layer="96" rot="R90"/>
+</instance>
+<instance part="S6" gate="1" x="15.24" y="66.04" smashed="yes">
+<attribute name="NAME" x="17.78" y="62.23" size="1.778" layer="95" rot="R90"/>
+<attribute name="VALUE" x="20.32" y="62.23" size="1.778" layer="96" rot="R90"/>
+</instance>
+<instance part="S7" gate="1" x="15.24" y="50.8" smashed="yes">
+<attribute name="NAME" x="17.78" y="46.99" size="1.778" layer="95" rot="R90"/>
+<attribute name="VALUE" x="20.32" y="46.99" size="1.778" layer="96" rot="R90"/>
+</instance>
+<instance part="S8" gate="1" x="15.24" y="30.48" smashed="yes">
+<attribute name="NAME" x="17.78" y="26.67" size="1.778" layer="95" rot="R90"/>
+<attribute name="VALUE" x="20.32" y="26.67" size="1.778" layer="96" rot="R90"/>
+</instance>
 </instances>
 <busses>
 </busses>
 <nets>
+<net name="N$1" class="0">
+<segment>
+<pinref part="S8" gate="1" pin="2"/>
+<pinref part="R4" gate="G$1" pin="1"/>
+<wire x1="15.24" y1="35.56" x2="25.4" y2="35.56" width="0.1524" layer="91"/>
+</segment>
+</net>
+<net name="N$2" class="0">
+<segment>
+<pinref part="S7" gate="1" pin="2"/>
+<pinref part="R3" gate="G$1" pin="1"/>
+<wire x1="15.24" y1="55.88" x2="27.94" y2="55.88" width="0.1524" layer="91"/>
+</segment>
+</net>
+<net name="N$3" class="0">
+<segment>
+<pinref part="S6" gate="1" pin="2"/>
+<pinref part="R2" gate="G$1" pin="1"/>
+<wire x1="15.24" y1="71.12" x2="25.4" y2="71.12" width="0.1524" layer="91"/>
+</segment>
+</net>
+<net name="N$4" class="0">
+<segment>
+<pinref part="S5" gate="1" pin="2"/>
+<pinref part="R1" gate="G$1" pin="1"/>
+<wire x1="15.24" y1="88.9" x2="25.4" y2="88.9" width="0.1524" layer="91"/>
+</segment>
+</net>
 </nets>
 </sheet>
@@
 packages will not be understood (or retained) with this version.
 </note>
+<note version="8.4" severity="warning">
+Since Version 8.4, EAGLE supports properties for SPICE simulation.
+Probes in schematics and SPICE mapping objects found in parts and library devices
+will not be understood with this version. Update EAGLE to the latest version
+for full support of SPICE simulation.
+</note>
 </compatibility>

Commit message: Updated PCB schematic
Parts:
- removed LED1, LED2, LED3: (no value), led:LED3MM
- removed R2: (no value), rcl:R-US_0309/12
- removed S7, S8: (no value), switch-dil:DS01E
- added ADLIGHTSWITCH, RESETBUTTON, SMARTCONTROLSWITCH: (no value), switch-dil:DS01E
- added G1: AB9V, battery:AB9V
- added G2: SL-340/P3.6V, battery:SL-340/P3.6V
- added LEDENGINE, LEDEXT, LEDINFO: (no value), led:LED3MM
- added U$1: NANO, Arduino-clone:NANO
Connections:
- new net N$10: LEDENGINE.A, U$1.D6
- new net N$11: LEDINFO.A, U$1.D7
- new net N$12: S5.2, U$1.RAW
- new net N$13: G1.-, G2.-, R1.2, R3.2, R4.2, U$1.GND
- new net N$14: R1.1, RESETBUTTON.2, U$1.D2
- new net N$9: ADLIGHTSWITCH.1, LEDEXT.A, RESETBUTTON.1, SMARTCONTROLSWITCH.1, U$1.5.5V
- net N$1: now also ADLIGHTSWITCH.2, U$1.D3; no longer S8.2
- net N$2: now also SMARTCONTROLSWITCH.2, U$1.D4; no longer S7.2
- net N$3: now also G2.+, S6.1; no longer R2.1, S6.2
- net N$4: now also G1.+, S5.1; no longer R1.1, S5.2
Other:
- moved on the sheet: R1, R3, R4, S5, S6

Commit message: Updated Board
Parts:
- added D1: (no value), diode:ZENER-DIODEP1-Z12
- added R2: (no value), rcl:R-US_0309/12
- added T1: 2N4923, transistor:2N4923
Connections:
- removed net N$13: G1.-, G2.-, R1.2, R3.2, R4.2, U$1.GND
- new net N$15: D1.C, R2.1, T1.B
- new net N$16: R2.2, S6.2, T1.C
- new net N$5: T1.E
- new net N$6: D1.A, G1.-, G2.-, LEDENGINE.C, LEDEXT.C, LEDINFO.C, R1.2, R3.2, R4.2, U$1.GND
Changed lines of the file:
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@@
 <part name="RESETBUTTON" library="switch-dil" library_urn="urn:adsk.eagle:library:375" deviceset="DS01E" device="" package3d_urn="urn:adsk.eagle:package:27201/2"/>
 <part name="R1" library="rcl" library_urn="urn:adsk.eagle:library:334" deviceset="R-US_" device="0309/12" package3d_urn="urn:adsk.eagle:package:23571/1"/>
+<part name="D1" library="diode" library_urn="urn:adsk.eagle:library:210" deviceset="ZENER-DIODE" device="P1-Z12" package3d_urn="urn:adsk.eagle:package:43340/1"/>
+<part name="R2" library="rcl" library_urn="urn:adsk.eagle:library:334" deviceset="R-US_" device="0309/12" package3d_urn="urn:adsk.eagle:package:23571/1"/>
+<part name="T1" library="transistor" library_urn="urn:adsk.eagle:library:402" deviceset="2N4923" device="" package3d_urn="urn:adsk.eagle:package:29898/1"/>
 </parts>
 <sheets>
 <sheet>
 <plain>
+<circle x="228.6" y="111.76" radius="5.6796125" width="0.1524" layer="94"/>
 </plain>
 <instances>
@@
 <attribute name="NAME" x="151.13" y="92.4814" size="1.778" layer="95" rot="R180"/>
 <attribute name="VALUE" x="151.13" y="97.282" size="1.778" layer="96" rot="R180"/>
+</instance>
+<instance part="D1" gate="G$1" x="205.74" y="101.6" smashed="yes" rot="R90">
+<attribute name="NAME" x="203.835" y="99.822" size="1.778" layer="95" rot="R90"/>
+<attribute name="VALUE" x="209.169" y="99.822" size="1.778" layer="96" rot="R90"/>
+</instance>
+<instance part="R2" gate="G$1" x="193.04" y="109.22" smashed="yes" rot="R180">
+<attribute name="NAME" x="196.85" y="107.7214" size="1.778" layer="95" rot="R180"/>
+<attribute name="VALUE" x="196.85" y="112.522" size="1.778" layer="96" rot="R180"/>
+</instance>
+<instance part="T1" gate="G$1" x="205.74" y="124.46" smashed="yes" rot="R90">
+<attribute name="NAME" x="198.12" y="114.3" size="1.778" layer="95" rot="R90"/>
+<attribute name="VALUE" x="200.66" y="114.3" size="1.778" layer="96" rot="R90"/>
 </instance>
 </instances>
@@
 </segment>
 </net>
-<net name="N$13" class="0">
-<segment>
+<net name="N$3" class="0">
+<segment>
+<pinref part="S6" gate="1" pin="1"/>
+<pinref part="G2" gate="G$1" pin="+"/>
+<wire x1="162.56" y1="124.46" x2="134.62" y2="124.46" width="0.1524" layer="91"/>
+</segment>
+</net>
+<net name="N$14" class="0">
+<segment>
+<pinref part="RESETBUTTON" gate="1" pin="2"/>
+<pinref part="R1" gate="G$1" pin="1"/>
+<wire x1="162.56" y1="93.98" x2="152.4" y2="93.98" width="0.1524" layer="91"/>
+<wire x1="162.56" y1="93.98" x2="162.56" y2="109.22" width="0.1524" layer="91"/>
+<junction x="162.56" y="93.98"/>
+<wire x1="162.56" y1="109.22" x2="58.42" y2="109.22" width="0.1524" layer="91"/>
+<wire x1="58.42" y1="109.22" x2="58.42" y2="147.32" width="0.1524" layer="91"/>
+<pinref part="U$1" gate="G$1" pin="D2"/>
+<wire x1="58.42" y1="147.32" x2="63.5" y2="147.32" width="0.1524" layer="91"/>
+</segment>
+</net>
+<net name="N$15" class="0">
+<segment>
+<pinref part="R2" gate="G$1" pin="1"/>
+<wire x1="198.12" y1="109.22" x2="205.74" y2="109.22" width="0.1524" layer="91"/>
+<pinref part="D1" gate="G$1" pin="C"/>
+<wire x1="205.74" y1="104.14" x2="205.74" y2="109.22" width="0.1524" layer="91"/>
+<pinref part="T1" gate="G$1" pin="B"/>
+<wire x1="205.74" y1="109.22" x2="205.74" y2="121.92" width="0.1524" layer="91"/>
+<junction x="205.74" y="109.22"/>
+</segment>
+</net>
+<net name="N$16" class="0">
+<segment>
+<pinref part="R2" gate="G$1" pin="2"/>
+<wire x1="187.96" y1="109.22" x2="187.96" y2="127" width="0.1524" layer="91"/>
+<pinref part="S6" gate="1" pin="2"/>
+<wire x1="187.96" y1="127" x2="187.96" y2="134.62" width="0.1524" layer="91"/>
+<wire x1="162.56" y1="134.62" x2="187.96" y2="134.62" width="0.1524" layer="91"/>
+<pinref part="T1" gate="G$1" pin="C"/>
+<wire x1="187.96" y1="127" x2="200.66" y2="127" width="0.1524" layer="91"/>
+<junction x="187.96" y="127"/>
+</segment>
+</net>
+<net name="N$5" class="0">
+<segment>
+<pinref part="T1" gate="G$1" pin="E"/>
+<wire x1="210.82" y1="127" x2="228.6" y2="127" width="0.1524" layer="91"/>
+<wire x1="228.6" y1="127" x2="228.6" y2="116.84" width="0.1524" layer="91"/>
+</segment>
+</net>
+<net name="N$6" class="0">
+<segment>
+<pinref part="D1" gate="G$1" pin="A"/>
+<wire x1="205.74" y1="99.06" x2="228.6" y2="99.06" width="0.1524" layer="91"/>
+<wire x1="228.6" y1="99.06" x2="228.6" y2="106.68" width="0.1524" layer="91"/>
+<wire x1="205.74" y1="99.06" x2="172.72" y2="99.06" width="0.1524" layer="91"/>
+<junction x="205.74" y="99.06"/>
+<wire x1="172.72" y1="99.06" x2="172.72" y2="114.3" width="0.1524" layer="91"/>
+<wire x1="172.72" y1="114.3" x2="114.3" y2="114.3" width="0.1524" layer="91"/>
 <pinref part="G1" gate="G$1" pin="-"/>
 <wire x1="116.84" y1="142.24" x2="106.68" y2="142.24" width="0.1524" layer="91"/>
@@
 <pinref part="G2" gate="G$1" pin="-"/>
 <wire x1="101.6" y1="154.94" x2="96.52" y2="154.94" width="0.1524" layer="91"/>
-<wire x1="124.46" y1="124.46" x2="106.68" y2="124.46" width="0.1524" layer="91"/>
+<wire x1="124.46" y1="124.46" x2="114.3" y2="124.46" width="0.1524" layer="91"/>
+<wire x1="114.3" y1="124.46" x2="106.68" y2="124.46" width="0.1524" layer="91"/>
 <wire x1="106.68" y1="124.46" x2="106.68" y2="142.24" width="0.1524" layer="91"/>
 <junction x="106.68" y="142.24"/>
@@
 <wire x1="142.24" y1="93.98" x2="101.6" y2="93.98" width="0.1524" layer="91"/>
 <junction x="101.6" y="93.98"/>
-</segment>
-</net>
-<net name="N$3" class="0">
-<segment>
-<pinref part="S6" gate="1" pin="1"/>
-<pinref part="G2" gate="G$1" pin="+"/>
-<wire x1="162.56" y1="124.46" x2="134.62" y2="124.46" width="0.1524" layer="91"/>
-</segment>
-</net>
-<net name="N$14" class="0">
-<segment>
-<pinref part="RESETBUTTON" gate="1" pin="2"/>
-<pinref part="R1" gate="G$1" pin="1"/>
-<wire x1="162.56" y1="93.98" x2="152.4" y2="93.98" width="0.1524" layer="91"/>
-<wire x1="162.56" y1="93.98" x2="162.56" y2="109.22" width="0.1524" layer="91"/>
-<junction x="162.56" y="93.98"/>
-<wire x1="162.56" y1="109.22" x2="58.42" y2="109.22" width="0.1524" layer="91"/>
-<wire x1="58.42" y1="109.22" x2="58.42" y2="147.32" width="0.1524" layer="91"/>
-<pinref part="U$1" gate="G$1" pin="D2"/>
-<wire x1="58.42" y1="147.32" x2="63.5" y2="147.32" width="0.1524" layer="91"/>
-</segment>
-</net>
+<wire x1="114.3" y1="114.3" x2="114.3" y2="124.46" width="0.1524" layer="91"/>
+<junction x="114.3" y="124.46"/>
+<wire x1="106.68" y1="124.46" x2="106.68" y2="101.6" width="0.1524" layer="91"/>
+<junction x="106.68" y="124.46"/>
+<wire x1="106.68" y1="101.6" x2="27.94" y2="101.6" width="0.1524" layer="91"/>
+<pinref part="LEDINFO" gate="G$1" pin="C"/>
+<pinref part="LEDENGINE" gate="G$1" pin="C"/>
+<wire x1="27.94" y1="127" x2="27.94" y2="139.7" width="0.1524" layer="91"/>
+<pinref part="LEDEXT" gate="G$1" pin="C"/>
+<wire x1="27.94" y1="152.4" x2="27.94" y2="139.7" width="0.1524" layer="91"/>
+<junction x="27.94" y="139.7"/>
+<wire x1="27.94" y1="101.6" x2="27.94" y2="127" width="0.1524" layer="91"/>
+<junction x="27.94" y="127"/>
+</segment>
+</net>
