File: ArduinoPCB.sch (EAGLE design)
At the start: 19 parts, among them T1 2N4923

Commit message: Updated PCB
Parts:
- removed D1: (no value), diode:ZENER-DIODEP1-Z12
- removed R2: (no value), rcl:R-US_0309/12
Connections:
- removed net N$15: D1.C, R2.1, T1.B
- net N$16: no longer R2.2
- net N$8: now also T1.B; no longer D1.A
Changed lines of the file:
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@@
 <part name="RESETBUTTON" library="switch-dil" library_urn="urn:adsk.eagle:library:375" deviceset="DS01E" device="" package3d_urn="urn:adsk.eagle:package:27201/2"/>
 <part name="R1" library="rcl" library_urn="urn:adsk.eagle:library:334" deviceset="R-US_" device="0309/12" package3d_urn="urn:adsk.eagle:package:23571/1"/>
-<part name="D1" library="diode" library_urn="urn:adsk.eagle:library:210" deviceset="ZENER-DIODE" device="P1-Z12" package3d_urn="urn:adsk.eagle:package:43340/1"/>
-<part name="R2" library="rcl" library_urn="urn:adsk.eagle:library:334" deviceset="R-US_" device="0309/12" package3d_urn="urn:adsk.eagle:package:23571/1"/>
 <part name="T1" library="transistor" library_urn="urn:adsk.eagle:library:402" deviceset="2N4923" device="" package3d_urn="urn:adsk.eagle:package:29898/1"/>
 <part name="LEDINFO1" library="led" library_urn="urn:adsk.eagle:library:259" deviceset="LED" device="3MM" package3d_urn="urn:adsk.eagle:package:15797/1"/>
@@
 <attribute name="NAME" x="151.13" y="92.4814" size="1.778" layer="95" rot="R180"/>
 <attribute name="VALUE" x="151.13" y="97.282" size="1.778" layer="96" rot="R180"/>
-</instance>
-<instance part="D1" gate="G$1" x="205.74" y="101.6" smashed="yes" rot="R90">
-<attribute name="NAME" x="203.835" y="99.822" size="1.778" layer="95" rot="R90"/>
-<attribute name="VALUE" x="209.169" y="99.822" size="1.778" layer="96" rot="R90"/>
-</instance>
-<instance part="R2" gate="G$1" x="193.04" y="109.22" smashed="yes" rot="R180">
-<attribute name="NAME" x="196.85" y="107.7214" size="1.778" layer="95" rot="R180"/>
-<attribute name="VALUE" x="196.85" y="112.522" size="1.778" layer="96" rot="R180"/>
 </instance>
 <instance part="T1" gate="G$1" x="205.74" y="124.46" smashed="yes" rot="R90">
@@
 </segment>
 </net>
-<net name="N$15" class="0">
-<segment>
-<pinref part="R2" gate="G$1" pin="1"/>
-<wire x1="198.12" y1="109.22" x2="205.74" y2="109.22" width="0.1524" layer="91"/>
-<pinref part="D1" gate="G$1" pin="C"/>
-<wire x1="205.74" y1="104.14" x2="205.74" y2="109.22" width="0.1524" layer="91"/>
-<pinref part="T1" gate="G$1" pin="B"/>
-<wire x1="205.74" y1="109.22" x2="205.74" y2="121.92" width="0.1524" layer="91"/>
-<junction x="205.74" y="109.22"/>
-</segment>
-</net>
 <net name="N$16" class="0">
 <segment>
-<pinref part="R2" gate="G$1" pin="2"/>
-<wire x1="187.96" y1="109.22" x2="187.96" y2="127" width="0.1524" layer="91"/>
 <pinref part="S6" gate="1" pin="2"/>
 <wire x1="187.96" y1="127" x2="187.96" y2="134.62" width="0.1524" layer="91"/>
@@
 <pinref part="T1" gate="G$1" pin="C"/>
 <wire x1="187.96" y1="127" x2="200.66" y2="127" width="0.1524" layer="91"/>
-<junction x="187.96" y="127"/>
 </segment>
 </net>
 <net name="N$8" class="0">
 <segment>
-<pinref part="D1" gate="G$1" pin="A"/>
+<wire x1="228.6" y1="99.06" x2="205.74" y2="99.06" width="0.1524" layer="91"/>
 <wire x1="205.74" y1="99.06" x2="172.72" y2="99.06" width="0.1524" layer="91"/>
 <wire x1="172.72" y1="99.06" x2="172.72" y2="114.3" width="0.1524" layer="91"/>
@@
 <junction x="27.94" y="127"/>
 <pinref part="LEDINFO1" gate="G$1" pin="C"/>
-<wire x1="205.74" y1="99.06" x2="228.6" y2="99.06" width="0.1524" layer="91"/>
 <wire x1="228.6" y1="99.06" x2="228.6" y2="106.68" width="0.1524" layer="91"/>
+<pinref part="T1" gate="G$1" pin="B"/>
+<wire x1="205.74" y1="121.92" x2="205.74" y2="99.06" width="0.1524" layer="91"/>
 <junction x="205.74" y="99.06"/>
 </segment>
