File: new_board.brd (EAGLE design)
At the start: 160 x 100 mm, 23 parts, among them J4 455-1750-1-ND, Q2 IRF3704L-V

Commit message: resize board
Parts:
- moved D2 39.4 mm to (35.6, 12.7)
- moved D3 39.4 mm to (24.1, 12.7)
- moved D5 39.4 mm to (44.5, 16.5)
- moved R1 39.4 mm to (12.7, 12.7)
- moved R2 39.4 mm to (10.2, 41.9)
- moved R3 39.4 mm to (3.81, 41.9)
- moved R4 39.4 mm to (21.6, 41.9)
- moved R5 39.4 mm to (16.5, 41.9)
- moved R7 39.4 mm to (35.6, 40.6)
- moved S1 39.4 mm to (29.2, 50.8)
- moved S2 39.4 mm to (19.1, 50.8)
- moved S3 39.4 mm to (7.62, 50.8)
- moved S4 39.4 mm to (15.2, 50.8)
- moved S5 39.4 mm to (39.4, 41.9)
- moved U$1 39.4 mm to (29.2, 27.9)
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Other:
- board size 160 x 100 mm -> 48.2 x 56.8 mm

Commit message: added ground and power planes, and changed resistor values/added resistor after the mosfet gate
Connections:
- net N$16 renamed 5V
Changed lines of the file:
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@@
 <wire x1="15.24" y1="24.13" x2="15.24" y2="22.86" width="0.1524" layer="21"/>
 <wire x1="17.78" y1="24.13" x2="17.78" y2="22.86" width="0.1524" layer="21"/>
+<dimension x1="0" y1="57.15" x2="48.26" y2="57.15" x3="24.13" y3="60.96" textsize="1.27" layer="20"/>
+<dimension x1="48.26" y1="57.15" x2="48.26" y2="0" x3="54.61" y3="28.575" textsize="1.27" layer="20"/>
 </plain>
 <attributes>
@@
 <wire x1="3.32603125" y1="10.2616" x2="4.9784" y2="10.2616" width="0.1524" layer="1"/>
 </signal>
-<signal name="N$16">
+<signal name="5V">
 <contactref element="S2" pad="1"/>
 <contactref element="U$1" pad="5V"/>
